File: pcb/OFT.kicad_sch (KiCad schematic)
At the start: 28 parts, among them J1 Conn_01x04_Pin, J2 IF-D92, J3 IF-E91A, U1 SN74LVC1G14, U4 SN74LVC1G14, U5 NE555D, U6 NE555D

Commit message: Change partlist vendors
Parts:
- J2, J3: Vendor DigiKey -> HTL; VendorId FB104-ND -> 103594
- U1, U4: Vendor DigiKey -> HTL; VendorId 296-11608-1-ND -> 103595
Changed lines of the file:
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@@
       (effects (font (size 1.27 1.27)) (justify left) hide)
     )
-    (property "Vendor" "DigiKey" (at 114.3 63.5 0)
-      (effects (font (size 1.27 1.27)) hide)
-    )
-    (property "VendorId" "296-11608-1-ND" (at 114.3 63.5 0)
+    (property "Vendor" "HTL" (at 114.3 63.5 0)
+      (effects (font (size 1.27 1.27)) hide)
+    )
+    (property "VendorId" "103595" (at 114.3 63.5 0)
       (effects (font (size 1.27 1.27)) hide)
     )
@@
       (effects (font (size 1.27 1.27)) (justify left) hide)
     )
-    (property "Vendor" "DigiKey" (at 119.38 134.62 0)
-      (effects (font (size 1.27 1.27)) hide)
-    )
-    (property "VendorId" "296-11608-1-ND" (at 119.38 134.62 0)
+    (property "Vendor" "HTL" (at 119.38 134.62 0)
+      (effects (font (size 1.27 1.27)) hide)
+    )
+    (property "VendorId" "103595" (at 119.38 134.62 0)
       (effects (font (size 1.27 1.27)) hide)
     )
@@
       (effects (font (size 1.27 1.27)) hide)
     )
-    (property "Vendor" "DigiKey" (at 87.63 67.31 0)
-      (effects (font (size 1.27 1.27)) hide)
-    )
-    (property "VendorId" "FB104-ND" (at 87.63 67.31 0)
+    (property "Vendor" "HTL" (at 87.63 67.31 0)
+      (effects (font (size 1.27 1.27)) hide)
+    )
+    (property "VendorId" "103594" (at 87.63 67.31 0)
       (effects (font (size 1.27 1.27)) hide)
     )
@@
       (effects (font (size 1.27 1.27)) hide)
     )
-    (property "Vendor" "DigiKey" (at 87.63 130.81 0)
-      (effects (font (size 1.27 1.27)) hide)
-    )
-    (property "VendorId" "FB104-ND" (at 87.63 130.81 0)
-      (effects (font (size 1.27 1.27)) hide)
-    )
+    (property "Vendor" "HTL" (at 87.63 130.81 0)
+      (effects (font (size 1.27 1.27)) hide)
+    )
+    (property "VendorId" "103594" (at 87.63 130.81 0)
+      (effects (font (size 1.27 1.27)) hide)
+    )

Commit message: Fix wrong vendor id
Parts:
- C6, C8: VendorId 100128 -> 103260
Changed lines of the file:
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@@
       (effects (font (size 1.27 1.27)) hide)
     )
-    (property "VendorId" "100128" (at 171.45 130.81 0)
+    (property "VendorId" "103260" (at 171.45 130.81 0)
       (effects (font (size 1.27 1.27)) hide)
     )
@@
       (effects (font (size 1.27 1.27)) hide)
     )
-    (property "VendorId" "100128" (at 171.45 80.01 0)
-      (effects (font (size 1.27 1.27)) hide)
-    )
+    (property "VendorId" "103260" (at 171.45 80.01 0)
+      (effects (font (size 1.27 1.27)) hide)
+    )
