File: pcb/OFT.kicad_sch (KiCad schematic)
At the start: 28 parts, among them J1 Conn_01x04_Pin, J2 IF-D92, J3 IF-E91A, U1 SN74LVC1G14, U4 SN74LVC1G14, U5 NE555D, U6 NE555D

Commit message: Rename fiducial reference
Parts:
- renumbered FID4 to FID1
Changed lines of the file:
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@@
 		(on_board yes)
 		(dnp no)
-		(property "Reference" "FID4"
+		(property "Reference" "FID1"
 			(at 151.13 175.26 0)
 			(effects
@@
 			(project "OFT"
 				(path "/9334361a-f7a5-4302-90e9-4b89798c8fc6"
-					(reference "FID4")
+					(reference "FID1")
 					(unit 1)
 				)
