File: pcb/OFT.kicad_pcb (KiCad board)
At the start: 2 copper layers, 26.7 x 25.4 mm, 28 parts, among them J1 Conn_01x04_Pin, J2 IF-D92, J3 IF-E91A, U1 SN74LVC1G14, U4 SN74LVC1G14, U5 NE555D, U6 NE555D

Commit message: Update to KiCAD 9
Parts:
- moved C1 0.39 mm to (155.3, 86.9)
- moved U1 0.18 mm to (158.3, 86.4)
- moved U4 0.18 mm to (158.3, 89.4)

Commit message: Optimize receiver load resistor
Parts:
- R1: value 2k2 -> 1k
Changed lines of the file:
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@@
 			)
 		)
-		(property "Value" "2k2"
+		(property "Value" "1k"
 			(at 3.3675 0 90)
 			(layer "B.Fab")
@@
 			)
 		)
-		(property "HTL" "102956"
+		(property "HTL" "102951"
 			(at 0 0 90)
 			(unlocked yes)
