File: pcb/OFT.kicad_pcb (KiCad board)
At the start: 2 copper layers, 26.7 x 25.4 mm, 28 parts, among them J1 Conn_01x04_Pin, J2 IF-D92, J3 IF-E91A, U1 SN74LVC1G14, U4 SN74LVC1G14, U5 NE555D, U6 NE555D

Commit message: Rename fiducial reference
Parts:
- renumbered FID4 to FID1
Changed lines of the file:
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@@
 		(layer "F.Cu")
 		(at 150.241 79.502)
-		(property "Reference" "FID4"
+		(property "Reference" "FID1"
 			(at 0 3.81 0)
 			(unlocked yes)
